File: hardware/retro-console-keychain.kicad_pcb (KiCad board)
At the start: 2 copper layers, 40 x 72 mm, 15 parts, among them J1 USB-C Power

Commit message: Polish retro console PCB artwork
Other:
- board size 40 x 72 mm -> 52 x 76 mm
- board text added: "BEEP"
- board text added: "POWER"
Changed lines of the file:
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@@
     (pad "2" smd roundrect (at 0.7875 0) (size 0.875 0.95) (layers "F.Cu" "F.Paste" "F.Mask") (net 10 "LED5") (pinfunction "A") (roundrect_rratio 0.25))
   )
-  (gr_line (start 62 34) (end 66 28) (stroke (width 0.12) (type solid)) (layer "Edge.Cuts") (tstamp "r0000000-0000-4000-8000-000000000001"))
-  (gr_line (start 66 28) (end 98 28) (stroke (width 0.12) (type solid)) (layer "Edge.Cuts") (tstamp "r0000000-0000-4000-8000-000000000002"))
-  (gr_line (start 98 28) (end 102 34) (stroke (width 0.12) (type solid)) (layer "Edge.Cuts") (tstamp "r0000000-0000-4000-8000-000000000003"))
-  (gr_line (start 102 34) (end 102 92) (stroke (width 0.12) (type solid)) (layer "Edge.Cuts") (tstamp "r0000000-0000-4000-8000-000000000004"))
-  (gr_line (start 102 92) (end 96 100) (stroke (width 0.12) (type solid)) (layer "Edge.Cuts") (tstamp "r0000000-0000-4000-8000-000000000005"))
-  (gr_line (start 96 100) (end 68 100) (stroke (width 0.12) (type solid)) (layer "Edge.Cuts") (tstamp "r0000000-0000-4000-8000-000000000006"))
-  (gr_line (start 68 100) (end 62 92) (stroke (width 0.12) (type solid)) (layer "Edge.Cuts") (tstamp "r0000000-0000-4000-8000-000000000007"))
-  (gr_line (start 62 92) (end 62 34) (stroke (width 0.12) (type solid)) (layer "Edge.Cuts") (tstamp "r0000000-0000-4000-8000-000000000008"))  (gr_rect (start 64 43) (end 76 56) (stroke (width 0.18) (type solid)) (fill none) (layer "F.SilkS") (tstamp "r1000000-0000-4000-8000-000000000001"))
+  (gr_line (start 56 34) (end 62 26) (stroke (width 0.12) (type solid)) (layer "Edge.Cuts") (tstamp "r0000000-0000-4000-8000-000000000001"))
+  (gr_line (start 62 26) (end 102 26) (stroke (width 0.12) (type solid)) (layer "Edge.Cuts") (tstamp "r0000000-0000-4000-8000-000000000002"))
+  (gr_line (start 102 26) (end 108 34) (stroke (width 0.12) (type solid)) (layer "Edge.Cuts") (tstamp "r0000000-0000-4000-8000-000000000003"))
+  (gr_line (start 108 34) (end 108 92) (stroke (width 0.12) (type solid)) (layer "Edge.Cuts") (tstamp "r0000000-0000-4000-8000-000000000004"))
+  (gr_line (start 108 92) (end 100 102) (stroke (width 0.12) (type solid)) (layer "Edge.Cuts") (tstamp "r0000000-0000-4000-8000-000000000005"))
+  (gr_line (start 100 102) (end 64 102) (stroke (width 0.12) (type solid)) (layer "Edge.Cuts") (tstamp "r0000000-0000-4000-8000-000000000006"))
+  (gr_line (start 64 102) (end 56 92) (stroke (width 0.12) (type solid)) (layer "Edge.Cuts") (tstamp "r0000000-0000-4000-8000-000000000007"))
+  (gr_line (start 56 92) (end 56 34) (stroke (width 0.12) (type solid)) (layer "Edge.Cuts") (tstamp "r0000000-0000-4000-8000-000000000008"))  (gr_rect (start 64 43) (end 76 56) (stroke (width 0.18) (type solid)) (fill none) (layer "F.SilkS") (tstamp "r1000000-0000-4000-8000-000000000001"))
   (gr_line (start 66 54) (end 68 52) (stroke (width 0.16) (type solid)) (layer "F.SilkS") (tstamp "r1000000-0000-4000-8000-000000000002"))
   (gr_line (start 68 52) (end 70 54) (stroke (width 0.16) (type solid)) (layer "F.SilkS") (tstamp "r1000000-0000-4000-8000-000000000003"))
@@
   (gr_circle (center 91 70) (end 93 70) (stroke (width 0.18) (type solid)) (fill none) (layer "F.SilkS") (tstamp "r1000000-0000-4000-8000-000000000009"))
   (gr_circle (center 86 77) (end 88 77) (stroke (width 0.18) (type solid)) (fill none) (layer "F.SilkS") (tstamp "r1000000-0000-4000-8000-000000000010"))
-(via (at 80.48 87.92) (size 0.6) (drill 0.3) (layers "F.Cu" "B.Cu") (net 2))
+  (gr_rect (start 58 39) (end 76 62) (stroke (width 0.24) (type solid)) (fill none) (layer "F.SilkS") (tstamp "r3000000-0000-4000-8000-000000000001"))
+  (gr_line (start 61 58) (end 65 54) (stroke (width 0.18) (type solid)) (layer "F.SilkS") (tstamp "r3000000-0000-4000-8000-000000000002"))
+  (gr_line (start 65 54) (end 68 58) (stroke (width 0.18) (type solid)) (layer "F.SilkS") (tstamp "r3000000-0000-4000-8000-000000000003"))
+  (gr_line (start 70 58) (end 73 54) (stroke (width 0.18) (type solid)) (layer "F.SilkS") (tstamp "r3000000-0000-4000-8000-000000000004"))
+  (gr_line (start 73 54) (end 75 58) (stroke (width 0.18) (type solid)) (layer "F.SilkS") (tstamp "r3000000-0000-4000-8000-000000000005"))
+  (gr_line (start 62 66) (end 72 66) (stroke (width 0.20) (type solid)) (layer "F.SilkS") (tstamp "r3000000-0000-4000-8000-000000000006"))
+  (gr_line (start 66 75) (end 66 89) (stroke (width 0.28) (type solid)) (layer "F.SilkS") (tstamp "r3000000-0000-4000-8000-000000000007"))
+  (gr_line (start 59 82) (end 73 82) (stroke (width 0.28) (type solid)) (layer "F.SilkS") (tstamp "r3000000-0000-4000-8000-000000000008"))
+  (gr_circle (center 100 70) (end 103 70) (stroke (width 0.24) (type solid)) (fill none) (layer "F.SilkS") (tstamp "r3000000-0000-4000-8000-000000000009"))
+  (gr_circle (center 95 80) (end 98 80) (stroke (width 0.24) (type solid)) (fill none) (layer "F.SilkS") (tstamp "r3000000-0000-4000-8000-000000000010"))
+  (gr_circle (center 101 87) (end 103 87) (stroke (width 0.18) (type solid)) (fill none) (layer "F.SilkS") (tstamp "r3000000-0000-4000-8000-000000000011"))
+  (gr_line (start 93 44) (end 104 44) (stroke (width 0.16) (type solid)) (layer "F.SilkS") (tstamp "r3000000-0000-4000-8000-000000000012"))
+  (gr_line (start 93 49) (end 101 49) (stroke (width 0.16) (type solid)) (layer "F.SilkS") (tstamp "r3000000-0000-4000-8000-000000000013"))
+  (gr_line (start 93 54) (end 104 54) (stroke (width 0.16) (type solid)) (layer "F.SilkS") (tstamp "r3000000-0000-4000-8000-000000000014"))
+  (gr_text "BEEP" (at 62 34 0) (layer "F.SilkS") (tstamp "r3000000-0000-4000-8000-000000000015") (effects (font (size 2 2) (thickness 0.25)) (justify left)))
+  (gr_text "POWER" (at 91 38 0) (layer "F.SilkS") (tstamp "r3000000-0000-4000-8000-000000000016") (effects (font (size 1.4 1.4) (thickness 0.18)) (justify left)))(via (at 80.48 87.92) (size 0.6) (drill 0.3) (layers "F.Cu" "B.Cu") (net 2))
   (via (at 83.52 87.92) (size 0.6) (drill 0.3) (layers "F.Cu" "B.Cu") (net 2))
   (via (at 80.6 81.2) (size 0.6) (drill 0.3) (layers "F.Cu" "B.Cu") (net 2))
